File: Hardware/rele wifi valensisi_ramos 6º5 v3.kicad_sch (KiCad schematic)
At the start: 45 parts, among them J1 relay-1, J2 relay-2, J3 relay-3, J4 relay-4, J5 entrada, J6 relay-1.1, J7 relay-2.2, J8 relay-3.3, J9 relay-4.4, K1 Relay_DPDT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

Commit message: Add files via upload
Parts:
- removed J1: relay-1, TerminalBlock:TerminalBlock_bornier-3_P5.08mm, symbol Connector:Screw_Terminal_01x03
- removed J2: relay-2, TerminalBlock:TerminalBlock_bornier-3_P5.08mm, symbol Connector:Screw_Terminal_01x03
- removed J3: relay-3, TerminalBlock:TerminalBlock_bornier-3_P5.08mm, symbol Connector:Screw_Terminal_01x03
- removed J4: relay-4, TerminalBlock:TerminalBlock_bornier-3_P5.08mm, symbol Connector:Screw_Terminal_01x03
- removed J5: entrada, TerminalBlock:TerminalBlock_MaiXu_MX126-5.0-02P_1x02_P5.00mm, symbol Connector:Screw_Terminal_01x02
- removed J6: relay-1.1, TerminalBlock:TerminalBlock_bornier-3_P5.08mm, symbol Connector:Screw_Terminal_01x03
- removed J7: relay-2.2, TerminalBlock:TerminalBlock_bornier-3_P5.08mm, symbol Connector:Screw_Terminal_01x03
- removed J8: relay-3.3, TerminalBlock:TerminalBlock_bornier-3_P5.08mm, symbol Connector:Screw_Terminal_01x03
- removed J9: relay-4.4, TerminalBlock:TerminalBlock_bornier-3_P5.08mm, symbol Connector:Screw_Terminal_01x03
- added D9: LED, LED_THT:LED_D5.0mm, symbol Device:LED
- added J1: entrada, symbol Connector:Screw_Terminal_01x02
- added J6: Screw_Terminal_01x16, TerminalBlock:TerminalBlock_MaiXu_MX126-5.0-16P_1x16_P5.00mm, symbol Connector:Screw_Terminal_01x16
- added R13: 470, Resistor_SMD:R_0805_2012Metric_Pad1.20x1.40mm_HandSolder, symbol Device:R
- added SW1: SW_DPST_x2, TerminalBlock:TerminalBlock_bornier-3_P5.08mm, symbol Switch:SW_DPST_x2
- D1, D2, D3, D4: footprint Diode_THT:D_DO-41_SOD81_P10.16mm_Horizontal -> Diode_SMD:D_SMA
- Q1, Q2, Q3, Q4: footprint Package_TO_SOT_THT:TO-92L_Inline -> Package_TO_SOT_THT:TO-92_Inline_Wide
Connections:
- net +12V: now also R13.1, SW1.2 (B)
- net COM-1: now also J6.14 (Pin_14)
- net COM-1.1: now also J6.15 (Pin_15)
- net COM-2: now also J6.10 (Pin_10)
- net COM-2.2: now also J6.11 (Pin_11)
- net COM-3: now also J6.6 (Pin_6)
- net COM-3.3: now also J6.7 (Pin_7)
- net COM-4: now also J6.2 (Pin_2)
- net COM-4.4: now also J6.3 (Pin_3)
- net GND: now also U7.38 (GND), D9.1 (K), J1.1 (Pin_1)
- net NO-1: now also J6.13 (Pin_13)
- net NO-1.1: now also J6.16 (Pin_16)
- net NO-2: now also J6.9 (Pin_9)
- net NO-2.2: now also J6.12 (Pin_12)
- net NO-3: now also J6.5 (Pin_5)
- net NO-3.3: now also J6.8 (Pin_8)
- net NO-4: now also J6.1 (Pin_1)
- net NO-4.4: now also J6.4 (Pin_4)
- net P16: now reaches U7.27 (IO16)
- net P16: now also R2.1
- net P17: now reaches U7.28 (IO17)
- net P17: now also R7.1
- net P4: no longer names the net of U7.26 (IO4)
- net P4: no longer R2.1
- net P5: no longer names the net of U7.29 (IO5)
- net P5: no longer R7.1
- new net: D9.2 (A), R13.2
- new net: J1.2 (Pin_2), SW1.1 (A)
Other:
- moved on the sheet: C10, C9, U6, U7
